File: control unit.kicad_sch (KiCad schematic)
At the start: 56 parts, among them CN1 10nF 10V, CN2 10nF 10V, IC2 STM32G431C6T6, J4 Conn_ST_STDC14, P1 USB_C_Plug_USB2.0, SW1 reset, U4 MCP1755ST-3302E/DB, Y1 16MHz

Commit message: added wire step
Parts:
- renumbered C41 to C53, C42 to C54, C43 to C55, C44 to C56, C45 to C57, C46 to C58, C47 to C59, C48 to C60, C49 to C61, C50 to C62, C51 to C63, C52 to C64
