File: esc.kicad_pcb (KiCad board)
At the start: 4 copper layers, 142 parts, among them CN1 10nF 10V, CN2 10nF 10V, IC1 DRV8300UDPWR, IC2 STM32G431C6T6, J1 Conn_01x02, J2 Conn_01x05, J4 Conn_ST_STDC14, Q1 60V 95A, Q2 60V 95A, Q3 60V 95A, Q4 60V 95A, Q5 60V 95A, Q6 60V 95A, SW1 reset, U1 AP63205WU, U2 LM317_SOT-223, U3 INA4180A4, U4 MCP1755ST-3302E/DB, Y1 16MHz

Commit message: pcb : finished mosfet and dclink, start gate driver
Parts:
- added C20: 10uF 50V, Capacitor_THT:C_Radial_D5.0mm_H11.0mm_P2.00mm, F.Cu at (95.9, 124.2)
- added C27: 10uF 50V, Capacitor_THT:C_Radial_D5.0mm_H11.0mm_P2.00mm, F.Cu at (102.3, 124.2)
- added C28: 10uF 50V, Capacitor_THT:C_Radial_D5.0mm_H11.0mm_P2.00mm, F.Cu at (108.7, 124.2)
- IC1, J1, R1, R10, R13, R14, R15, R16, R2, R3, R4, R7, R8, R9, U2: moved to B.Cu
- moved R2 209.5 mm to (133.7, 79.3), turned to -90 degrees
- moved R1 209.3 mm to (133.7, 60.8), turned to 90 degrees
- moved U2 208.5 mm to (140.7, 124.4), turned to 90 degrees
- moved R3 207.2 mm to (131.3, 60.8), turned to 90 degrees
- moved R4 207.0 mm to (131.3, 79.3), turned to -90 degrees
- moved IC1 206.0 mm to (147.4, 89.7), turned to 180 degrees
- moved R14 193.0 mm to (133.5, 123.3), turned to -90 degrees
- moved R16 189.5 mm to (131.3, 123.3), turned to -90 degrees
- moved R13 189.1 mm to (133.5, 104.8), turned to 90 degrees
- moved R15 185.9 mm to (131.3, 104.8), turned to 90 degrees
- moved R8 164.2 mm to (133.5, 101.3), turned to -90 degrees
- moved R7 161.8 mm to (133.5, 82.8), turned to 90 degrees
- moved R10 161.1 mm to (131.3, 101.3), turned to -90 degrees
- moved R9 159.1 mm to (131.3, 82.8), turned to 90 degrees
- moved C29 141.1 mm to (63.9, 108.7)
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Routing:
- net /VBAT_{fused}: track 23.7 -> 47.1 mm
- net /power/half_bridge1/G_{L}: track 0.00 -> 20.2 mm, vias 0 -> 1
- net /power/half_bridge3/G_{L}: track 0.00 -> 20.0 mm, vias 0 -> 1
- net /power/half_bridge2/G_{L}: track 0.00 -> 20.0 mm, vias 0 -> 1
- net /power/half_bridge2/G_{H}: track 0.00 -> 12.5 mm
- net /power/half_bridge1/G_{H}: track 0.00 -> 12.5 mm
- net /power/half_bridge3/G_{H}: track 0.00 -> 12.4 mm
- net /PHASE3: track 15.0 -> 8.90 mm
- net /power/half_bridge1/GND_{SHUNT}: track 6.80 -> 10.1 mm, vias 0 -> 10
- net /power/half_bridge2/GND_{SHUNT}: track 6.80 -> 10.1 mm, vias 0 -> 10
- net /power/half_bridge3/GND_{SHUNT}: track 6.80 -> 10.1 mm, vias 0 -> 10
- net /PHASE1: track 15.1 -> 18.2 mm
- net /PHASE2: track 15.2 -> 18.2 mm
- net PGND: vias 0 -> 24
- added copper zone on B.Cu, net /PHASE1
- added copper zone on In1.Cu, net /PHASE1
- added copper zone on In2.Cu, net /PHASE1
- added copper zone on B.Cu, net /PHASE2
- added copper zone on In1.Cu, net /PHASE2
- added copper zone on In2.Cu, net /PHASE2
- added copper zone on B.Cu, net /PHASE3
- added copper zone on In1.Cu, net /PHASE3
- added copper zone on In2.Cu, net /PHASE3
- added copper zone on B.Cu, net /VBAT_{fused}
- added copper zone on In1.Cu, net /VBAT_{fused}
- added copper zone on In2.Cu, net /VBAT_{fused}
- added copper zone on In2.Cu, net /power/half_bridge1/GND_{SHUNT}
- added copper zone on In2.Cu, net /power/half_bridge2/GND_{SHUNT}
- added copper zone on In2.Cu, net /power/half_bridge3/GND_{SHUNT}
Other:
- board outline added: 80 x 75 mm

Commit message: added wire step
Parts:
- removed the C20 at (95.9, 124.2)
- added C12: 10uF 50V, Capacitor_THT:C_Radial_D5.0mm_H11.0mm_P2.00mm, F.Cu at (95.9, 124.2)
- added C14: 470nF 35V, Capacitor_SMD:C_0603_1608Metric, B.Cu at (115.7, 68.1)
- added C15: 470nF 35V, Capacitor_SMD:C_0603_1608Metric, B.Cu at (115.7, 71.8)
- added C16: 470nF 35V, Capacitor_SMD:C_0603_1608Metric, B.Cu at (115.7, 69.9)
- added C24: 10uF 50V, Capacitor_THT:C_Radial_D5.0mm_H11.0mm_P2.00mm, F.Cu at (102.3, 124.2)
- added C26: 470nF 35V, Capacitor_SMD:C_0603_1608Metric, B.Cu at (115.6, 89.9)
- added C36: 10uF 50V, Capacitor_THT:C_Radial_D5.0mm_H11.0mm_P2.00mm, F.Cu at (108.7, 124.2)
- added C38: 470nF 35V, Capacitor_SMD:C_0603_1608Metric, B.Cu at (115.6, 111.8)
- added C39: 470nF 35V, Capacitor_SMD:C_0603_1608Metric, B.Cu at (115.6, 113.8)
- added C40: 470nF 35V, Capacitor_SMD:C_0603_1608Metric, B.Cu at (115.6, 115.8)
- added J5: Conn_01x01, MountingHole:MountingHole_3mm_Pad_Via, B.Cu at (128.0, 71.5)
- added J6: Conn_01x01, MountingHole:MountingHole_3mm_Pad_Via, B.Cu at (128.0, 93.5)
- added J7: Conn_01x01, MountingHole:MountingHole_3mm_Pad_Via, B.Cu at (128.0, 115.5)
- C27, C28: value 10uF 50V -> 470nF 35V; footprint Capacitor_THT:C_Radial_D5.0mm_H11.0mm_P2.00mm -> Capacitor_SMD:C_0603_1608Metric; moved to B.Cu
- C41: renamed from C29; moved to B.Cu
- C42: renamed from C30; moved to B.Cu
- C43: renamed from C31; moved to B.Cu
- C44: renamed from C32; moved to B.Cu
- C45: renamed from C33; moved to B.Cu
- C46: renamed from C34; moved to B.Cu
- C47: renamed from C35; moved to B.Cu
- D2, J2, R19, R20, VR1: moved to B.Cu
- moved J2 155.4 mm to (136.4, 75.5), turned to 90 degrees
- moved TP7 90.6 mm to (166.2, 102.2)
- moved C42 84.1 mm to (145.9, 94.8)
- moved C43 83.0 mm to (145.9, 98.3)
- moved C41 82.9 mm to (145.9, 96.5)
- moved C45 78.5 mm to (133.5, 90.2), turned to -90 degrees
- moved C46 78.4 mm to (133.5, 93.5), turned to -90 degrees
- moved C47 78.4 mm to (133.5, 96.7), turned to -90 degrees
- moved R20 74.5 mm to (142.4, 110.0), turned to 180 degrees
- moved R19 74.5 mm to (142.4, 108.1), turned to 180 degrees
- moved C44 73.5 mm to (144.9, 102.4)
- moved VR1 65.3 mm to (137.7, 110.1), turned to 90 degrees
- moved D2 64.2 mm to (142.4, 111.8), turned to 180 degrees
- moved C27 34.9 mm to (115.6, 91.9), turned to 180 degrees
- moved C28 31.1 mm to (115.6, 93.9), turned to 180 degrees
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- renumbered C12 to C10, C9 to C11, C10 to C13, C13 to C17, C14 to C18, C15 to C19, C19 to C20, C16 to C21, C20 to C22, C17 to C23, C18 to C25, C21 to C29, C22 to C30, C23 to C31, C27 to C32, C24 to C33, C28 to C34, C25 to C35, C26 to C37, C36 to C48, C37 to C49, C38 to C50, C39 to C51, C40 to C52, C41 to C53, C42 to C54, C43 to C55, C44 to C56, C45 to C57, C46 to C58, C47 to C59, C48 to C60, C49 to C61, C50 to C62, C51 to C63, C52 to C64, C11 to C8, C8 to C9
Connections:
- C45 pad 2: /PHASE1 -> /PHASE2
- C46 pad 2: /PHASE2 -> /PHASE1
- IC1 pad 1: /control unit/GATE_H1_{filt} -> /control unit/GATE_H2_{filt}
- IC1 pad 10: /power/GATE_{L2} -> /power/GATE_{L1}
- IC1 pad 11: /power/GATE_{L1} -> /power/GATE_{L2}
- IC1 pad 15: /PHASE2 -> /PHASE1
- IC1 pad 16: /power/GATE_{H2} -> /power/GATE_{H1}
- IC1 pad 18: /PHASE1 -> /PHASE2
- IC1 pad 19: /power/GATE_{H1} -> /power/GATE_{H2}
- IC1 pad 2: /control unit/GATE_H2_{filt} -> /control unit/GATE_H1_{filt}
- IC1 pad 4: /control unit/GATE_L1_{filt} -> /control unit/GATE_L2_{filt}
- IC1 pad 5: /control unit/GATE_L2_{filt} -> /control unit/GATE_L1_{filt}
- U2 pad 3: +24V -> /VBAT_{fused}
Routing:
- net /power/GATE_{H1}: track 0.00 -> 34.3 mm
- net /power/GATE_{L3}: track 0.00 -> 32.0 mm, vias 0 -> 2
- net /power/GATE_{L1}: track 0.00 -> 23.5 mm, vias 0 -> 4
- net /PHASE3: track 8.90 -> 32.1 mm, vias 0 -> 2
- net /PHASE1: track 18.2 -> 39.6 mm, vias 0 -> 2
- net Net-(IC1-GVDD): track 0.00 -> 19.3 mm
- net /power/GATE_{H3}: track 0.00 -> 14.0 mm
- net /VBAT_{fused}: track 47.1 -> 59.3 mm
- net /power/GATE_{H2}: track 0.00 -> 10.0 mm
- net Net-(U2-ADJ): track 0.00 -> 6.86 mm
- net /power/GATE_{L2}: track 0.00 -> 5.64 mm
- net /PHASE2: track 18.2 -> 23.6 mm
- net /power/half_bridge2/G_{L}: track 20.0 -> 23.5 mm
- net /power/half_bridge3/G_{L}: track 20.0 -> 23.5 mm
- net /power/half_bridge1/G_{L}: track 20.2 -> 23.6 mm
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- added copper zone on B.Cu, net PGND
- added copper zone on F.Cu, net PGND
- added copper zone on In1.Cu, net PGND
- added copper zone on In2.Cu, net PGND
