File: power.kicad_sch (KiCad schematic)
At the start: 24 parts, among them IC1 DRV8300UDPWR, U2 LM317_SOT-223, U3 INA4180A4

Commit message: added wire step
Parts:
- renumbered C29 to C41, C30 to C42, C31 to C43, C32 to C44, C33 to C45, C34 to C46, C35 to C47, C36 to C48, C37 to C49, C38 to C50, C39 to C51, C40 to C52
Connections:
- net +24V is gone; now on net VBAT: U2.3 (VI)
- net GATE_H1_{filt}: now also IC1.2 (INHB); no longer IC1.1 (INHA)
- net GATE_H2_{filt}: now also IC1.1 (INHA); no longer IC1.2 (INHB)
- net GATE_L1_{filt}: now also IC1.5 (INLB); no longer IC1.4 (INLA)
- net GATE_L2_{filt}: now also IC1.4 (INLA); no longer IC1.5 (INLB)
- net GATE_{H1}: now also IC1.16 (GHB); no longer IC1.19 (GHA)
- net GATE_{H2}: now also IC1.19 (GHA); no longer IC1.16 (GHB)
- net GATE_{L1}: now also IC1.10 (GLB); no longer IC1.11 (GLA)
- net GATE_{L2}: now also IC1.11 (GLA); no longer IC1.10 (GLB)
- net PHASE1: now also C46.2, IC1.15 (SHB); no longer C45.2, IC1.18 (SHA)
- net PHASE2: now also C45.2, IC1.18 (SHA); no longer C46.2, IC1.15 (SHB)
